File: Sterownik_Podlewania/1.1/Przyciski.kicad_sch (KiCad schematic)
At the start: 12 parts, among them SW3 SW_Push_Dual_x2, SW4 SW_Push_Dual_x2, SW5 SW_Push_Dual_x2, SW6 SW_Push_Dual_x2

Commit message: Poprawiono błędy połączeń SDA,SCL, dodno drugą magistralę I2C, pociągnięcie nowych ścieżek
Parts:
- SW1: renamed from SW4; footprint Button_Switch_SMD:SW_SPST_TL3305A -> Button_Switch_THT:SW_PUSH_6mm
- SW2: renamed from SW3; footprint Button_Switch_SMD:SW_SPST_TL3305A -> Button_Switch_THT:SW_PUSH_6mm
- SW3: renamed from SW5; footprint Button_Switch_SMD:SW_SPST_TL3305A -> Button_Switch_THT:SW_PUSH_6mm
- SW4: renamed from SW6; footprint Button_Switch_SMD:SW_SPST_TL3305A -> Button_Switch_THT:SW_PUSH_6mm
- renumbered C3 to C10, C6 to C7, C5 to C8, C4 to C9, R31 to R17, R28 to R18, R27 to R21, R26 to R22
Changed lines of the file:
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@@
 		(dnp no)
 		(fields_autoplaced yes)
-		(property "Reference" "R26"
+		(property "Reference" "R22"
 			(at 104.14 77.4699 0)
 			(effects
@@
 			(project ""
 				(path "/a66bdf1f-0e2a-4cc5-beb1-605f2a3b9885/98590924-e867-4033-87b1-a5aeee05e762"
-					(reference "R26")
+					(reference "R22")
 					(unit 1)
 				)
@@
 		(dnp no)
 		(fields_autoplaced yes)
-		(property "Reference" "R28"
+		(property "Reference" "R18"
 			(at 198.12 77.4699 0)
 			(effects
@@
 			(project "Sterownik_Podlewania V1.1"
 				(path "/a66bdf1f-0e2a-4cc5-beb1-605f2a3b9885/98590924-e867-4033-87b1-a5aeee05e762"
-					(reference "R28")
+					(reference "R18")
 					(unit 1)
 				)
@@
 		(dnp no)
 		(fields_autoplaced yes)
-		(property "Reference" "R31"
+		(property "Reference" "R17"
 			(at 252.73 76.1999 0)
 			(effects
@@
 			(project "Sterownik_Podlewania V1.1"
 				(path "/a66bdf1f-0e2a-4cc5-beb1-605f2a3b9885/98590924-e867-4033-87b1-a5aeee05e762"
-					(reference "R31")
+					(reference "R17")
 					(unit 1)
 				)
@@
 		(dnp no)
 		(fields_autoplaced yes)
-		(property "Reference" "C6"
+		(property "Reference" "C7"
 			(at 254 96.5199 0)
 			(effects
@@
 			(project "Sterownik_Podlewania V1.1"
 				(path "/a66bdf1f-0e2a-4cc5-beb1-605f2a3b9885/98590924-e867-4033-87b1-a5aeee05e762"
-					(reference "C6")
+					(reference "C7")
 					(unit 1)
 				)
@@
 		(dnp no)
 		(fields_autoplaced yes)
-		(property "Reference" "SW6"
+		(property "Reference" "SW4"
 			(at 238.76 80.01 0)
 			(effects
@@
 			)
 		)
-		(property "Footprint" "Button_Switch_SMD:SW_SPST_TL3305A"
+		(property "Footprint" "Button_Switch_THT:SW_PUSH_6mm"
 			(at 238.76 82.55 0)
 			(effects
@@
 			(project "Sterownik_Podlewania V1.1"
 				(path "/a66bdf1f-0e2a-4cc5-beb1-605f2a3b9885/98590924-e867-4033-87b1-a5aeee05e762"
-					(reference "SW6")
+					(reference "SW4")
 					(unit 1)
 				)
@@
 		(dnp no)
 		(fields_autoplaced yes)
-		(property "Reference" "SW5"
+		(property "Reference" "SW3"
 			(at 184.15 81.28 0)
 			(effects
@@
 			)
 		)
-		(property "Footprint" "Button_Switch_SMD:SW_SPST_TL3305A"
+		(property "Footprint" "Button_Switch_THT:SW_PUSH_6mm"
 			(at 184.15 83.82 0)
 			(effects
@@
 			(project "Sterownik_Podlewania V1.1"
 				(path "/a66bdf1f-0e2a-4cc5-beb1-605f2a3b9885/98590924-e867-4033-87b1-a5aeee05e762"
-					(reference "SW5")
+					(reference "SW3")
 					(unit 1)
 				)
@@
 		(dnp no)
 		(fields_autoplaced yes)
-		(property "Reference" "C3"
+		(property "Reference" "C10"
 			(at 105.41 97.7899 0)
 			(effects
@@
 			(project ""
 				(path "/a66bdf1f-0e2a-4cc5-beb1-605f2a3b9885/98590924-e867-4033-87b1-a5aeee05e762"
-					(reference "C3")
+					(reference "C10")
 					(unit 1)
 				)
@@
 		(dnp no)
 		(fields_autoplaced yes)
-		(property "Reference" "C5"
+		(property "Reference" "C8"
 			(at 199.39 97.7899 0)
 			(effects
@@
 			(project "Sterownik_Podlewania V1.1"
 				(path "/a66bdf1f-0e2a-4cc5-beb1-605f2a3b9885/98590924-e867-4033-87b1-a5aeee05e762"
-					(reference "C5")
+					(reference "C8")
 					(unit 1)
 				)
@@
 		(dnp no)
 		(fields_autoplaced yes)
-		(property "Reference" "R27"
+		(property "Reference" "R21"
 			(at 151.13 77.4699 0)
 			(effects
@@
 			(project "Sterownik_Podlewania V1.1"
 				(path "/a66bdf1f-0e2a-4cc5-beb1-605f2a3b9885/98590924-e867-4033-87b1-a5aeee05e762"
-					(reference "R27")
+					(reference "R21")
 					(unit 1)
 				)
@@
 		(dnp no)
 		(fields_autoplaced yes)
-		(property "Reference" "C4"
+		(property "Reference" "C9"
 			(at 152.4 97.7899 0)
 			(effects
@@
 			(project "Sterownik_Podlewania V1.1"
 				(path "/a66bdf1f-0e2a-4cc5-beb1-605f2a3b9885/98590924-e867-4033-87b1-a5aeee05e762"
-					(reference "C4")
+					(reference "C9")
 					(unit 1)
 				)
@@
 		(dnp no)
 		(fields_autoplaced yes)
-		(property "Reference" "SW3"
+		(property "Reference" "SW2"
 			(at 137.16 81.28 0)
 			(effects
@@
 			)
 		)
-		(property "Footprint" "Button_Switch_SMD:SW_SPST_TL3305A"
+		(property "Footprint" "Button_Switch_THT:SW_PUSH_6mm"
 			(at 137.16 83.82 0)
 			(effects
@@
 			(project "Sterownik_Podlewania V1.1"
 				(path "/a66bdf1f-0e2a-4cc5-beb1-605f2a3b9885/98590924-e867-4033-87b1-a5aeee05e762"
-					(reference "SW3")
+					(reference "SW2")
 					(unit 1)
 				)
@@
 		(dnp no)
 		(fields_autoplaced yes)
-		(property "Reference" "SW4"
+		(property "Reference" "SW1"
 			(at 90.17 81.28 0)
 			(effects
@@
 			)
 		)
-		(property "Footprint" "Button_Switch_SMD:SW_SPST_TL3305A"
+		(property "Footprint" "Button_Switch_THT:SW_PUSH_6mm"
 			(at 90.17 83.82 0)
 			(effects
@@
 			(project ""
 				(path "/a66bdf1f-0e2a-4cc5-beb1-605f2a3b9885/98590924-e867-4033-87b1-a5aeee05e762"
-					(reference "SW4")
-					(unit 1)
-				)
+					(reference "SW1")
+					(unit 1)
+				)

Commit message: Usunięcie zewnętrzego zasilania 12 i stabilizatora napięcia, korekcja zasilania wzmacniacz operacyjny moduł zasilania
Parts:
- renumbered C10 to C3, C9 to C4, C8 to C5, C7 to C6, R22 to R18, R21 to R19, R18 to R20, R17 to R21, SW1 to SW3, SW2 to SW4, SW3 to SW5, SW4 to SW6
Changed lines of the file:
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@@
 		(dnp no)
 		(fields_autoplaced yes)
-		(property "Reference" "R22"
+		(property "Reference" "R18"
 			(at 104.14 77.4699 0)
 			(effects
@@
 			(project ""
 				(path "/a66bdf1f-0e2a-4cc5-beb1-605f2a3b9885/98590924-e867-4033-87b1-a5aeee05e762"
-					(reference "R22")
+					(reference "R18")
 					(unit 1)
 				)
@@
 		(dnp no)
 		(fields_autoplaced yes)
-		(property "Reference" "#PWR067"
+		(property "Reference" "#PWR073"
 			(at 250.19 73.66 0)
 			(effects
@@
 			(project "Sterownik_Podlewania V1.1"
 				(path "/a66bdf1f-0e2a-4cc5-beb1-605f2a3b9885/98590924-e867-4033-87b1-a5aeee05e762"
-					(reference "#PWR067")
+					(reference "#PWR073")
 					(unit 1)
 				)
@@
 		(dnp no)
 		(fields_autoplaced yes)
-		(property "Reference" "R18"
+		(property "Reference" "R20"
 			(at 198.12 77.4699 0)
 			(effects
@@
 			(project "Sterownik_Podlewania V1.1"
 				(path "/a66bdf1f-0e2a-4cc5-beb1-605f2a3b9885/98590924-e867-4033-87b1-a5aeee05e762"
-					(reference "R18")
+					(reference "R20")
 					(unit 1)
 				)
@@
 		(dnp no)
 		(fields_autoplaced yes)
-		(property "Reference" "R17"
+		(property "Reference" "R21"
 			(at 252.73 76.1999 0)
 			(effects
@@
 			(project "Sterownik_Podlewania V1.1"
 				(path "/a66bdf1f-0e2a-4cc5-beb1-605f2a3b9885/98590924-e867-4033-87b1-a5aeee05e762"
-					(reference "R17")
+					(reference "R21")
 					(unit 1)
 				)
@@
 		(dnp no)
 		(fields_autoplaced yes)
-		(property "Reference" "C7"
+		(property "Reference" "C6"
 			(at 254 96.5199 0)
 			(effects
@@
 			(project "Sterownik_Podlewania V1.1"
 				(path "/a66bdf1f-0e2a-4cc5-beb1-605f2a3b9885/98590924-e867-4033-87b1-a5aeee05e762"
-					(reference "C7")
+					(reference "C6")
 					(unit 1)
 				)
@@
 		(dnp no)
 		(fields_autoplaced yes)
-		(property "Reference" "SW4"
+		(property "Reference" "SW6"
 			(at 238.76 80.01 0)
 			(effects
@@
 			(project "Sterownik_Podlewania V1.1"
 				(path "/a66bdf1f-0e2a-4cc5-beb1-605f2a3b9885/98590924-e867-4033-87b1-a5aeee05e762"
-					(reference "SW4")
+					(reference "SW6")
 					(unit 1)
 				)
@@
 		(dnp no)
 		(fields_autoplaced yes)
-		(property "Reference" "#PWR063"
+		(property "Reference" "#PWR069"
 			(at 148.59 74.93 0)
 			(effects
@@
 			(project "Sterownik_Podlewania V1.1"
 				(path "/a66bdf1f-0e2a-4cc5-beb1-605f2a3b9885/98590924-e867-4033-87b1-a5aeee05e762"
-					(reference "#PWR063")
+					(reference "#PWR069")
 					(unit 1)
 				)
@@
 		(dnp no)
 		(fields_autoplaced yes)
-		(property "Reference" "#PWR062"
+		(property "Reference" "#PWR068"
 			(at 119.38 110.49 0)
 			(effects
@@
 			(project "Sterownik_Podlewania V1.1"
 				(path "/a66bdf1f-0e2a-4cc5-beb1-605f2a3b9885/98590924-e867-4033-87b1-a5aeee05e762"
-					(reference "#PWR062")
+					(reference "#PWR068")
 					(unit 1)
 				)
@@
 		(dnp no)
 		(fields_autoplaced yes)
-		(property "Reference" "#PWR064"
+		(property "Reference" "#PWR070"
 			(at 166.37 110.49 0)
 			(effects
@@
 			(project "Sterownik_Podlewania V1.1"
 				(path "/a66bdf1f-0e2a-4cc5-beb1-605f2a3b9885/98590924-e867-4033-87b1-a5aeee05e762"
-					(reference "#PWR064")
+					(reference "#PWR070")
 					(unit 1)
 				)
@@
 		(dnp no)
 		(fields_autoplaced yes)
-		(property "Reference" "SW3"
+		(property "Reference" "SW5"
 			(at 184.15 81.28 0)
 			(effects
@@
 			(project "Sterownik_Podlewania V1.1"
 				(path "/a66bdf1f-0e2a-4cc5-beb1-605f2a3b9885/98590924-e867-4033-87b1-a5aeee05e762"
-					(reference "SW3")
+					(reference "SW5")
 					(unit 1)
 				)
@@
 		(dnp no)
 		(fields_autoplaced yes)
-		(property "Reference" "C10"
+		(property "Reference" "C3"
 			(at 105.41 97.7899 0)
 			(effects
@@
 			(project ""
 				(path "/a66bdf1f-0e2a-4cc5-beb1-605f2a3b9885/98590924-e867-4033-87b1-a5aeee05e762"
-					(reference "C10")
+					(reference "C3")
 					(unit 1)
 				)
@@
 		(dnp no)
 		(fields_autoplaced yes)
-		(property "Reference" "#PWR066"
+		(property "Reference" "#PWR072"
 			(at 220.98 109.22 0)
 			(effects
@@
 			(project "Sterownik_Podlewania V1.1"
 				(path "/a66bdf1f-0e2a-4cc5-beb1-605f2a3b9885/98590924-e867-4033-87b1-a5aeee05e762"
-					(reference "#PWR066")
+					(reference "#PWR072")
 					(unit 1)
 				)
@@
 		(dnp no)
 		(fields_autoplaced yes)
-		(property "Reference" "#PWR060"
+		(property "Reference" "#PWR066"
 			(at 72.39 110.49 0)
 			(effects
@@
 			(project ""
 				(path "/a66bdf1f-0e2a-4cc5-beb1-605f2a3b9885/98590924-e867-4033-87b1-a5aeee05e762"
-					(reference "#PWR060")
+					(reference "#PWR066")
 					(unit 1)
 				)
@@
 		(dnp no)
 		(fields_autoplaced yes)
-		(property "Reference" "C8"
+		(property "Reference" "C5"
 			(at 199.39 97.7899 0)
 			(effects
@@
 			(project "Sterownik_Podlewania V1.1"
 				(path "/a66bdf1f-0e2a-4cc5-beb1-605f2a3b9885/98590924-e867-4033-87b1-a5aeee05e762"
-					(reference "C8")
+					(reference "C5")
 					(unit 1)
 				)
@@
 		(dnp no)
 		(fields_autoplaced yes)
-		(property "Reference" "#PWR065"
+		(property "Reference" "#PWR071"
 			(at 195.58 74.93 0)
 			(effects
@@
 			(project "Sterownik_Podlewania V1.1"
 				(path "/a66bdf1f-0e2a-4cc5-beb1-605f2a3b9885/98590924-e867-4033-87b1-a5aeee05e762"
-					(reference "#PWR065")
+					(reference "#PWR071")
 					(unit 1)
 				)
@@
 		(dnp no)
 		(fields_autoplaced yes)
-		(property "Reference" "R21"
+		(property "Reference" "R19"
 			(at 151.13 77.4699 0)
 			(effects
@@
 			(project "Sterownik_Podlewania V1.1"
 				(path "/a66bdf1f-0e2a-4cc5-beb1-605f2a3b9885/98590924-e867-4033-87b1-a5aeee05e762"
-					(reference "R21")
+					(reference "R19")
 					(unit 1)
 				)
@@
 		(dnp no)
 		(fields_autoplaced yes)
-		(property "Reference" "#PWR061"
+		(property "Reference" "#PWR067"
 			(at 101.6 74.93 0)
 			(effects
@@
 			(project ""
 				(path "/a66bdf1f-0e2a-4cc5-beb1-605f2a3b9885/98590924-e867-4033-87b1-a5aeee05e762"
-					(reference "#PWR061")
+					(reference "#PWR067")
 					(unit 1)
 				)
@@
 		(dnp no)
 		(fields_autoplaced yes)
-		(property "Reference" "C9"
+		(property "Reference" "C4"
 			(at 152.4 97.7899 0)
 			(effects
@@
 			(project "Sterownik_Podlewania V1.1"
 				(path "/a66bdf1f-0e2a-4cc5-beb1-605f2a3b9885/98590924-e867-4033-87b1-a5aeee05e762"
-					(reference "C9")
+					(reference "C4")
 					(unit 1)
 				)
@@
 		(dnp no)
 		(fields_autoplaced yes)
-		(property "Reference" "SW2"
+		(property "Reference" "SW4"
 			(at 137.16 81.28 0)
 			(effects
@@
 			(project "Sterownik_Podlewania V1.1"
 				(path "/a66bdf1f-0e2a-4cc5-beb1-605f2a3b9885/98590924-e867-4033-87b1-a5aeee05e762"
-					(reference "SW2")
+					(reference "SW4")
 					(unit 1)
 				)
@@
 		(dnp no)
 		(fields_autoplaced yes)
-		(property "Reference" "SW1"
+		(property "Reference" "SW3"
 			(at 90.17 81.28 0)
 			(effects
@@
 			(project ""
 				(path "/a66bdf1f-0e2a-4cc5-beb1-605f2a3b9885/98590924-e867-4033-87b1-a5aeee05e762"
-					(reference "SW1")
-					(unit 1)
-				)
+					(reference "SW3")
+					(unit 1)
+				)

Commit message: Werja plików podesłana Mariuszkowi, dodane opisy i numeracja poprawna dla steronwika, w module poprawniono opis złącze ethernet
Parts:
- renumbered C3 to C10, C6 to C7, C5 to C8, C4 to C9, R21 to R18, R20 to R19, R19 to R20, R18 to R21, SW4 to SW1, SW3 to SW2, SW5 to SW3, SW6 to SW4
Changed lines of the file:
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@@
 		(dnp no)
 		(fields_autoplaced yes)
-		(property "Reference" "R18"
+		(property "Reference" "R21"
 			(at 104.14 77.4699 0)
 			(effects
@@
 			(project ""
 				(path "/a66bdf1f-0e2a-4cc5-beb1-605f2a3b9885/98590924-e867-4033-87b1-a5aeee05e762"
-					(reference "R18")
+					(reference "R21")
 					(unit 1)
 				)
@@
 		(dnp no)
 		(fields_autoplaced yes)
-		(property "Reference" "R20"
+		(property "Reference" "R19"
 			(at 198.12 77.4699 0)
 			(effects
@@
 			(project "Sterownik_Podlewania V1.1"
 				(path "/a66bdf1f-0e2a-4cc5-beb1-605f2a3b9885/98590924-e867-4033-87b1-a5aeee05e762"
-					(reference "R20")
+					(reference "R19")
 					(unit 1)
 				)
@@
 		(dnp no)
 		(fields_autoplaced yes)
-		(property "Reference" "R21"
+		(property "Reference" "R18"
 			(at 252.73 76.1999 0)
 			(effects
@@
 			(project "Sterownik_Podlewania V1.1"
 				(path "/a66bdf1f-0e2a-4cc5-beb1-605f2a3b9885/98590924-e867-4033-87b1-a5aeee05e762"
-					(reference "R21")
+					(reference "R18")
 					(unit 1)
 				)
@@
 		(dnp no)
 		(fields_autoplaced yes)
-		(property "Reference" "C6"
+		(property "Reference" "C7"
 			(at 254 96.5199 0)
 			(effects
@@
 			(project "Sterownik_Podlewania V1.1"
 				(path "/a66bdf1f-0e2a-4cc5-beb1-605f2a3b9885/98590924-e867-4033-87b1-a5aeee05e762"
-					(reference "C6")
+					(reference "C7")
 					(unit 1)
 				)
@@
 		(dnp no)
 		(fields_autoplaced yes)
-		(property "Reference" "SW6"
+		(property "Reference" "SW4"
 			(at 238.76 80.01 0)
 			(effects
@@
 			(project "Sterownik_Podlewania V1.1"
 				(path "/a66bdf1f-0e2a-4cc5-beb1-605f2a3b9885/98590924-e867-4033-87b1-a5aeee05e762"
-					(reference "SW6")
+					(reference "SW4")
 					(unit 1)
 				)
@@
 		(dnp no)
 		(fields_autoplaced yes)
-		(property "Reference" "SW5"
+		(property "Reference" "SW3"
 			(at 184.15 81.28 0)
 			(effects
@@
 			(project "Sterownik_Podlewania V1.1"
 				(path "/a66bdf1f-0e2a-4cc5-beb1-605f2a3b9885/98590924-e867-4033-87b1-a5aeee05e762"
-					(reference "SW5")
+					(reference "SW3")
 					(unit 1)
 				)
@@
 		(dnp no)
 		(fields_autoplaced yes)
-		(property "Reference" "C3"
+		(property "Reference" "C10"
 			(at 105.41 97.7899 0)
 			(effects
@@
 			(project ""
 				(path "/a66bdf1f-0e2a-4cc5-beb1-605f2a3b9885/98590924-e867-4033-87b1-a5aeee05e762"
-					(reference "C3")
+					(reference "C10")
 					(unit 1)
 				)
@@
 		(dnp no)
 		(fields_autoplaced yes)
-		(property "Reference" "C5"
+		(property "Reference" "C8"
 			(at 199.39 97.7899 0)
 			(effects
@@
 			(project "Sterownik_Podlewania V1.1"
 				(path "/a66bdf1f-0e2a-4cc5-beb1-605f2a3b9885/98590924-e867-4033-87b1-a5aeee05e762"
-					(reference "C5")
+					(reference "C8")
 					(unit 1)
 				)
@@
 		(dnp no)
 		(fields_autoplaced yes)
-		(property "Reference" "R19"
+		(property "Reference" "R20"
 			(at 151.13 77.4699 0)
 			(effects
@@
 			(project "Sterownik_Podlewania V1.1"
 				(path "/a66bdf1f-0e2a-4cc5-beb1-605f2a3b9885/98590924-e867-4033-87b1-a5aeee05e762"
-					(reference "R19")
+					(reference "R20")
 					(unit 1)
 				)
@@
 		(dnp no)
 		(fields_autoplaced yes)
-		(property "Reference" "C4"
+		(property "Reference" "C9"
 			(at 152.4 97.7899 0)
 			(effects
@@
 			(project "Sterownik_Podlewania V1.1"
 				(path "/a66bdf1f-0e2a-4cc5-beb1-605f2a3b9885/98590924-e867-4033-87b1-a5aeee05e762"
-					(reference "C4")
+					(reference "C9")
 					(unit 1)
 				)
@@
 		(dnp no)
 		(fields_autoplaced yes)
-		(property "Reference" "SW4"
+		(property "Reference" "SW1"
 			(at 137.16 81.28 0)
 			(effects
@@
 			(project "Sterownik_Podlewania V1.1"
 				(path "/a66bdf1f-0e2a-4cc5-beb1-605f2a3b9885/98590924-e867-4033-87b1-a5aeee05e762"
-					(reference "SW4")
+					(reference "SW1")
 					(unit 1)
 				)
@@
 		(dnp no)
 		(fields_autoplaced yes)
-		(property "Reference" "SW3"
+		(property "Reference" "SW2"
 			(at 90.17 81.28 0)
 			(effects
@@
 			(project ""
 				(path "/a66bdf1f-0e2a-4cc5-beb1-605f2a3b9885/98590924-e867-4033-87b1-a5aeee05e762"
-					(reference "SW3")
-					(unit 1)
-				)
+					(reference "SW2")
+					(unit 1)
+				)
